Commit message: Phase 1 Checkpoint 1 Task 3: Add Sensor Plugins Completed

File: my_rb1_description/urdf/my_rb1_robot.urdf (robot description, URDF)
Before this commit: robot robot, 7 links, 6 joints
Links:
- link base_footprint: mass 10 -> 15
- link base_link: mass 10 -> 5
- link left_wheel: geometry collision cylinder length=0.025 radius=0.05; visual cylinder length=0.025 radius=0.05
- link right_wheel: geometry collision cylinder length=0.025 radius=0.05; visual cylinder length=0.025 radius=0.05
Joints:
- joint base_to_back_caster: origin xyz=0.1 0.0 -0.15 -> xyz=0.1 0.0 -0.15 rpy=0 0 0
- joint base_to_base_footprint: origin xyz=0.0 0.0 -0.15 -> xyz=0.0 0.0 -0.15 rpy=0 0 0
- joint base_to_front_laser: type continuous -> fixed
- joint base_to_right_wheel: origin xyz=0.0 -0.2 -0.15 -> xyz=0.0 -0.2 -0.15 rpy=0 0 0

Commit message: Phase 1 Checkpoint 1 Task1, Task2, and Task3 Completed; Comments Resolved and Ready for Re-evaluation

File: my_rb1_description/urdf/my_rb1_robot.urdf (robot description, URDF)
Before this commit: robot robot, 7 links, 6 joints
Links:
- link back_caster: geometry collision sphere radius=0.02; collision sphere radius=0.04
- link base_footprint: mass 15 -> 21
- link base_link: mass 5 -> None
- link front_caster: geometry collision sphere radius=0.02; collision sphere radius=0.04
- link front_laser: geometry collision cylinder length=0.05 radius=0.025; visual cylinder length=0.05 radius=0.025
- link left_wheel: geometry collision cylinder length=0.05 radius=0.05; visual cylinder length=0.05 radius=0.05
- link right_wheel: geometry collision cylinder length=0.05 radius=0.05; visual cylinder length=0.05 radius=0.05
Joints:
- joint base_to_back_caster: origin xyz=0.1 0.0 -0.15 rpy=0 0 0 -> xyz=-0.1 0.0 -0.15 rpy=0 0 0
- joint base_to_base_footprint: type continuous -> fixed
- joint base_to_front_caster: origin xyz=-0.1 0.0 -0.15 rpy=0 0 0 -> xyz=0.1 0.0 -0.15 rpy=0 0 0
